File: 01_KiCAD/00_schematics/STM32 Nucleo RS232 & RS485 Expansion Board (ST Zio Compatible) V2/RX_TX_LED.kicad_sch (KiCad schematic)
At the start: 22 parts, among them J4 TX_LED, J5 RX_LED, U3 SN74LVC2G14DBV

Commit message: Updated PCB
Updated PCB with components layout and routing tracks.
Connections:
- net RX_RC: now reaches C24.2, C25.1, D6.2 (A), R16.2, U3.3 (2A)
Changed lines of the file:
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@@
+		)
+	)
+	(label "RX_RC"
+		(at 91.44 113.03 0)
+		(effects
+			(font
+				(size 1.016 1.016)
+				(color 221 133 0 1)
+			)
+			(justify left bottom)
 		)
 	)

Commit message: Complete redesign
Redesigned the complete board. Added hardware termination jumpers for 1120R resistors for RS485. Changes footprint, package size and simplified values between capacitors.
Still need to re-route the entire board :-(
Parts:
- renumbered C20 to C23, C21 to C24, C22 to C25, C24 to C26, C25 to C27, D3 to D2, D4 to D3, D5 to D4, D6 to D5, J4 to J8, J5 to J9, R10 to R12, R11 to R13, R12 to R14, R13 to R15, R14 to R16, R15 to R17, R16 to R18, R17 to R19, R18 to R20, R19 to R21, U3 to U4

Commit message: Small changes to schematics & PCB work
Made some minor adjustments to the schematics, updated the PCB accordingly.
Placed all the components on the board and did some of the routing.
Updated the 3D models of all the components.
Parts:
- C25: footprint PCM_SparkFun-Capacitor:C_0603_1608Metric -> Capacitor_SMD:C_0805_2012Metric
Changed lines of the file:
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@@
 			)
 		)
-		(property "Footprint" "PCM_SparkFun-Capacitor:C_0603_1608Metric"
+		(property "Footprint" "Capacitor_SMD:C_0805_2012Metric"
 			(at 133.35 76.2 0)
 			(effects
