File: 01_KiCAD/00_schematics/STM32 Nucleo RS232 & RS485 Expansion Board (ST Zio Compatible) V2/RX_TX_LED.kicad_sch (KiCad schematic)
At the start: 22 parts, among them J8 TX LED, J9 RX LED, U4 SN74LVC2G14DBV

Commit message: Final revision checkup
After BOM-update and corrected some footprints and package sizes for resistors and capacitors, updated the PCB to "HW REV A0.2" as final PCB layout. Need to run DRC check before final approval.
Parts:
- C23, C26: footprint PCM_SparkFun-Capacitor:C_0603_1608Metric -> Capacitor_SMD:C_0805_2012Metric; Dielectric X7R 20% -> X7R; MPN CC0603KRX7R9BB104 -> 08055C474JAT2A; Manufacturer YAGEO -> Kyocera AVX; Mouser PN (none) -> 581-08055C474JAT2A; Package 0603 -> 0805; Tolerance 20% -> 5%; Voltage 25V -> 50V
- C24, C27: footprint PCM_SparkFun-Capacitor:C_0603_1608Metric -> Capacitor_SMD:C_0805_2012Metric; Dielectric X7R 5% -> X7R; LCSC C91183 -> C2167095; MPN CC0603JRX7R9BB104 -> C0805C104J5RACTU; Manufacturer YAGEO -> KEMET; Mouser PN (none) -> 80-C0805C104J5R; Package 0603 -> 0805; Tolerance 20% -> 5%; Voltage 25V -> 50V
- C25: Dielectric X7R 5% -> X7R; LCSC C91183 -> C2167095; MPN CC0603JRX7R9BB104 -> C0805C104J5RACTU; Manufacturer YAGEO -> KEMET; Mouser PN (none) -> 80-C0805C104J5R; Package 0603 -> 0805; Tolerance 20% -> 5%; Voltage 25V -> 50V
- D2, D5: Mouser PN (none) -> 511-BAT54JFILM; Voltage (none) -> 40V
- D3: Color green -> Green; Mouser PN (none) -> 743-IN-S63AT5G; Voltage (none) -> 2,7V
- D4: Color amber -> Amber; Mouser PN (none) -> 743-IN-S63AT5A; Voltage (none) -> 2,0V
- J8, J9: LCSC C6631883 -> C5714562; Mouser PN (none) -> 200-HTSW10307GS
- R12, R17: LCSC C22548 -> C6113732; MPN RC0603FR-071KL -> AC0603FR-7W1KL; Mouser PN (none) -> 603-AC0603FR-7W1KL
- R13, R18: LCSC C114660 -> C227908; MPN RC0603FR-07150KL -> AC0603FR-07453KL; Mouser PN (none) -> 603-AC0603FR-07453KL
- R14, R21: LCSC C105881 -> C513549; MPN RC0603FR-07330RL -> AC0603FR-7W330RL; Mouser PN (none) -> 603-AC0603FR-7W330RL
- R15, R19: LCSC C105578 -> C20142017; MPN RC0603FR-071ML -> AC0603FR-7W1ML; Mouser PN (none) -> 603-AC0603FR-7W1ML
- R16: LCSC C22548 -> C227973; MPN RC0603FR-071KL -> AC0603FR-07590RL; Mouser PN (none) -> 603-AC0603FR-07590RL
- R20: LCSC C227580 -> C227579; MPN AC0603FR-07137RL -> AC0603FR-07137KL; Mouser PN (none) -> 603-AC0603FR-07137KL
- U4: LCSC (none) -> C12401; MPN (none) -> SN74LVC2G14DBVR; Manufacturer (none) -> TI; Mouser PN (none) -> 595-SN74LVC2G14DBVR; Package (none) -> SOT-23-6; Type (none) -> SMD
