File: 01_KiCAD/00_schematics/STM32 Nucleo RS232 & RS485 Expansion Board (ST Zio Compatible) V2/STM32 Nucleo RS232 & RS485 Expansion Board (ST Zio Compatible) V2.kicad_pcb (KiCad board)
At the start: 4 copper layers, 72 x 133.4 mm, 187 parts, among them CN10 Conn_02x17_Odd_Even, CN7 Conn_02x10_Odd_Even, CN8 Conn_02x08_Odd_Even, CN9 Conn_02x15_Odd_Even, J1 HD-A(Y), J10 SW_ENA, J11 MODE0, J12 MODE1, J13 MODE2, J14 DIR, J15 TERM_TX, J16 TERM_RX, J17 SLR, J2 HD-B(Z), J3 TERM (A/B), J4 TERM (Y/Z), J5 1190299, J6 CONN D-SUB PLUG 9POS TH, J7 TCVR_PWR, J8 TX_LED, J9 RX_LED, U1 TLV77518PDBVR, U2 TPS2117DRLR, U3 THVD4431RHAR, U4 SN74LVC2G14DBV, U5 SN74LVC245ADBR, U6 SN74LVC14ADR, U7 SN74LVC14ADR, U8 SN74LVC2G14DBV

Commit message: Small changes to schematics & PCB work
Made some minor adjustments to the schematics, updated the PCB accordingly.
Placed all the components on the board and did some of the routing.
Updated the 3D models of all the components.
Parts:
- removed TP31: GND, 5006_Black:KEYSTONE_5006
- C25, C28, C29, C30, C31: footprint PCM_SparkFun-Capacitor:C_0603_1608Metric -> Capacitor_SMD:C_0805_2012Metric
- TP2: value 5V0_IN -> 5V0 IN
- TP3: value 3V3_LDO -> 3V3 LDO
- TP5: value 3V3_IN -> 3V3 IN
- TP6: value 3V3_SYS -> 3V3 SYS
- moved C30 216.9 mm to (65.8, 120.9)
- moved C29 208.4 mm to (55.5, 121.5), turned to 180 degrees
- moved TP16 203.8 mm to (93.5, 77.2)
- moved TP13 201.3 mm to (93.5, 71.2)
- moved C28 195.1 mm to (70.4, 96.3), turned to -90 degrees
- moved TP10 189.8 mm to (93.5, 65.2)
- moved U8 167.3 mm to (75.1, 127.5)
- moved R45 160.3 mm to (88.0, 160.7), turned to 0 degrees
- moved D11 160.2 mm to (83.3, 164.3)
- moved R43 159.6 mm to (73.3, 160.7), turned to 0 degrees
- moved D9 159.5 mm to (68.6, 164.4)
- moved D12 159.2 mm to (85.3, 164.3)
- moved R30 159.2 mm to (90.7, 160.7), turned to 0 degrees
- moved R41 158.7 mm to (58.4, 160.7), turned to 0 degrees
- moved D10 158.5 mm to (70.6, 164.4)
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Connections:
- C20 pad 1: Net-(U3-C1-) -> Net-(U3-C2-)
- C20 pad 2: Net-(U3-C2-) -> Net-(U3-C2+)
- C21 pad 2: Net-(U3-C2+) -> Net-(U3-C1-)
- R26 pad 1: MCU_OE -> Net-(J10-Pin_2)
Routing:
- net Net-(J10-Pin_2): track 0.00 -> 157.0 mm
- net 3V3_SYS: track 19.8 -> 95.6 mm, vias 10 -> 50
- net Net-(D14-K): track 0.00 -> 73.9 mm
- net MODE2: track 21.7 -> 95.5 mm, vias 2 -> 4
- net Net-(D12-K): track 0.00 -> 73.8 mm, vias 0 -> 2
- net MCU_OE: track 0.00 -> 73.6 mm
- net Net-(D11-K): track 0.00 -> 68.1 mm, vias 0 -> 2
- net Net-(D13-K): track 0.00 -> 65.7 mm
- net GND: track 32.9 -> 98.4 mm, vias 16 -> 72
- net MODE1: track 18.3 -> 83.8 mm
- net MODE0: track 17.5 -> 78.4 mm
- net Net-(D8-K): track 0.00 -> 57.7 mm
- net Net-(D9-K): track 0.00 -> 56.7 mm
- net Net-(D10-K): track 0.00 -> 55.9 mm, vias 0 -> 2
- net SLR: track 15.6 -> 69.2 mm
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