File: 01_KiCAD/00_schematics/STM32 Nucleo RS232 & RS485 Expansion Board (ST Zio Compatible) V2/STM32 Nucleo RS232 & RS485 Expansion Board (ST Zio Compatible) V2.kicad_sch (KiCad schematic)
At the start: 22 parts

Commit message: Final revision checkup
After BOM-update and corrected some footprints and package sizes for resistors and capacitors, updated the PCB to "HW REV A0.2" as final PCB layout. Need to run DRC check before final approval.
Parts:
- TP10, TP19, TP30: footprint 5122_Blue:KEYSTONE_5122 -> 5121_Green:KEYSTONE_5121; LCSC (none) -> C5272789; MPN (none) -> 5121; Manufacturer (none) -> Keystone Electronics§; Mouser PN (none) -> 534-5121; Package None -> Through Hole,P=2.54mm; Type (none) -> THT
- TP11, TP14: LCSC (none) -> C238128; MPN (none) -> 5014; Manufacturer (none) -> Keystone Electronics§; Mouser PN (none) -> 534-5014; Package NON STANDARD-1 Keystone -> Through Hole,P=2.54mm; Type (none) -> THT
- TP12, TP15, TP23, TP25, TP27: footprint 5121_Green:KEYSTONE_5121 -> 5122_Blue:KEYSTONE_5122; LCSC (none) -> C5272796; MPN (none) -> 5122; Manufacturer (none) -> Keystone Electronics§; Mouser PN (none) -> 534-5122; Package None -> Through Hole,P=2.54mm; Type (none) -> THT
- TP13, TP16, TP24, TP26, TP28: LCSC (none) -> C5272796; MPN (none) -> 5122; Manufacturer (none) -> Keystone Electronics§; Mouser PN (none) -> 534-5122; Package None -> Through Hole,P=2.54mm; Type (none) -> THT
- TP17, TP20: LCSC (none) -> C2906767; MPN (none) -> 5013; Manufacturer (none) -> Keystone Electronics§; Mouser PN (none) -> 534-5013; Package NON STANDARD-1 Keystone -> Through Hole,P=2.54mm; Type (none) -> THT
- TP18, TP21, TP9: LCSC (none) -> C5272789; MPN (none) -> 5121; Manufacturer (none) -> Keystone Electronics§; Mouser PN (none) -> 534-5121; Package None -> Through Hole,P=2.54mm; Type (none) -> THT
- TP22, TP29: LCSC (none) -> C2906764; MPN (none) -> 5006; Manufacturer (none) -> Keystone Electronics; Mouser PN (none) -> 534-5006; Package NON STANDARD-1 Keystone -> Through Hole,P=2.54mm; Type (none) -> THT
